Commit message: random positioning of the goal marker with readl CAD robot

File: src/four_wheel_robot/description/gazebo_control.xacro (robot description, xacro)
@@ -19,6 +19,8 @@
         <wheel_separation>0.85</wheel_separation>
         <wheel_diameter>0.20</wheel_diameter>
-        <max_wheel_torque>8.0</max_wheel_torque>
-        <max_wheel_acceleration>1.5</max_wheel_acceleration>
+        <max_wheel_torque>30.0</max_wheel_torque>
+        <max_wheel_acceleration>30.0</max_wheel_acceleration>
+        <max_linear_speed>2.0</max_linear_speed>
+        <max_angular_speed>2.0</max_angular_speed>
         <command_topic>cmd_vel</command_topic>
         <odometry_topic>odom</odometry_topic>

File: src/four_wheel_robot/description/robot_core.xacro (robot description, xacro)
@@ -75,4 +75,5 @@
         <origin xyz="-0.3 -0.425 0" rpy="0 0 0" />
         <axis xyz="0 1 0" />
+        <!--<dynamics damping="0.2" friction="0.05"/>-->
     </joint>
     <link name="right_back_wheel">
@@ -90,5 +91,5 @@
             </geometry>
         </collision>
-        <xacro:inertial_cylinder mass="0.1" length="0.05" radius="0.1">
+        <xacro:inertial_cylinder mass="0.5" length="0.05" radius="0.1">
             <origin xyz="0 0 0" rpy="0 0 0"/>
         </xacro:inertial_cylinder>
@@ -97,5 +98,5 @@
         <material> Gazebo/Blue </material>
         <mu1>1.0</mu1><mu2>1.0</mu2>
-        <kp>1e6</kp><kd>1</kd>
+        <!--<kp>1e6</kp><kd>1</kd>-->
     </gazebo>
     <!-- LEFT BACK WHEEL LINK-->
@@ -120,5 +121,5 @@
             </geometry>
         </collision>
-        <xacro:inertial_cylinder mass="0.1" length="0.05" radius="0.1">
+        <xacro:inertial_cylinder mass="0.5" length="0.05" radius="0.1">
             <origin xyz="0 0 0" rpy="0 0 0"/>
         </xacro:inertial_cylinder>
@@ -127,5 +128,5 @@
         <material> Gazebo/Blue </material>
         <mu1>1.0</mu1><mu2>1.0</mu2>
-        <kp>1e6</kp><kd>1</kd>
+        <!--<kp>1e6</kp><kd>1</kd>-->
     </gazebo>
     <!-- RIGHT FRONT WHEEL LINK-->
@@ -150,5 +151,5 @@
             </geometry>
         </collision>
-        <xacro:inertial_cylinder mass="0.1" length="0.05" radius="0.1">
+        <xacro:inertial_cylinder mass="0.5" length="0.05" radius="0.1">
             <origin xyz="0 0 0" rpy="0 0 0"/>
         </xacro:inertial_cylinder>
@@ -157,5 +158,5 @@
         <material> Gazebo/Blue </material>
         <mu1>1.0</mu1><mu2>1.0</mu2>
-        <kp>1e6</kp><kd>1</kd>
+        <!--<kp>1e6</kp><kd>1</kd>-->
     </gazebo>
     <!-- LEFT FRONT WHEEL LINK-->
@@ -180,5 +181,5 @@
             </geometry>
         </collision>
-        <xacro:inertial_cylinder mass="0.1" length="0.05" radius="0.1">
+        <xacro:inertial_cylinder mass="0.5" length="0.05" radius="0.1">
             <origin xyz="0 0 0" rpy="0 0 0"/>
         </xacro:inertial_cylinder>
@@ -187,5 +188,5 @@
         <material> Gazebo/Blue </material>
         <mu1>1.0</mu1><mu2>1.0</mu2>
-        <kp>1e6</kp><kd>1</kd>
+        <!--<kp>1e6</kp><kd>1</kd>-->
     </gazebo>
     <!-- HANDLE MIDDLE LINK-->
