Commit message: Static Obsatcles added

File: src/my_robot_description/models/my_robot_description/depth_camera.xacro (robot description, xacro)
@@ -29,5 +29,5 @@
     <parent link="depth_camera_back_link"/>
     <child link="left_camera_link"/>
-    <origin xyz="0.0058 -0.036 0" rpy="0 0 0"/> <!-- Rotate to length along x (forward), baseline along y -->
+    <origin xyz="0.0058 0.036 0" rpy="0 0 0"/> <!-- Rotate to length along x (forward), baseline along y -->
   </joint>
   <link name="left_camera_link">
@@ -61,17 +61,24 @@
         <clip>
           <near>0.02</near>
-          <far>50.0</far>
+          <far>10.0</far>
         </clip>
-        <!--<noise>
-          <type>gaussian</type>
-          <mean>0.0</mean>
-          <stddev>0.01</stddev>
-        </noise>-->
       </camera>
       <plugin name="left_camera_controller" filename="libgazebo_ros_camera.so">
         <ros>
-          <namespace>/follower_robot</namespace>
+          <namespace>/follower_robot/depth_cam</namespace>
+          <qos>
+            <topic name="/follower_robot/depth_cam/left/image_raw">
+                <publisher>
+                    <reliability>reliable</reliability>
+                </publisher>
+            </topic>
+            <topic name="/follower_robot/depth_cam/left/camera_info">
+                <publisher>
+                    <reliability>reliable</reliability>
+                </publisher>
+            </topic>
+          </qos>
         </ros>
-        <camera_name>depth_cam/left</camera_name>
+        <camera_name>left</camera_name>
         <frame_name>left_camera_link_optical</frame_name>
         <!--<focal_length>1424.1969168622516</focal_length>
@@ -94,5 +101,5 @@
     <parent link="depth_camera_back_link"/>
     <child link="right_camera_link"/>
-    <origin xyz="0.0058 0.036 0" rpy="0 0 0"/> <!-- Rotate to length along x (forward), baseline along y -->
+    <origin xyz="0.0058 -0.036 0" rpy="0 0 0"/> <!-- Rotate to length along x (forward), baseline along y -->
   </joint>
   <link name="right_camera_link">
@@ -126,17 +133,24 @@
         <clip>
           <near>0.02</near>
-          <far>50.0</far>
+          <far>10.0</far>
         </clip>
-        <!--<noise>
-          <type>gaussian</type>
-          <mean>0.0</mean>
-          <stddev>0.01</stddev>
-        </noise>-->
       </camera>
       <plugin name="right_camera_controller" filename="libgazebo_ros_camera.so">
         <ros>
-          <namespace>/follower_robot</namespace>
+          <namespace>/follower_robot/depth_cam</namespace>
+          <qos>
+            <topic name="/follower_robot/depth_cam/right/image_raw">
+                <publisher>
+                    <reliability>reliable</reliability>
+                </publisher>
+            </topic>
+            <topic name="/follower_robot/depth_cam/right/camera_info">
+                <publisher>
+                    <reliability>reliable</reliability>
+                </publisher>
+            </topic>
+          </qos>
         </ros>
-        <camera_name>depth_cam/right</camera_name>  <!-- Sets prefix for topics: /depth_cam/right/image_raw and /depth_cam/right/camera_info -->
+        <camera_name>right</camera_name>  <!-- Sets prefix for topics: /depth_cam/right/image_raw and /depth_cam/right/camera_info -->
         <frame_name>right_camera_link_optical</frame_name>
         <!--<focal_length>1424.1969168622516</focal_length>
@@ -144,5 +158,5 @@
         <cy>615.3056335449219</cy>
         <cx_prime>812.6941986083984</cx_prime>-->
-        <hack_baseline>-0.071727</hack_baseline>
+        <hack_baseline>0.071727</hack_baseline>
       </plugin>
     </sensor>
@@ -155,8 +169,3 @@
   </joint>
   <link name="right_camera_link_optical"/>
-  <plugin name="clock_sync" filename="libgazebo_ros_clock.so">
-    <ros>
-      <namespace>/</namespace>
-    </ros>
-  </plugin>
 </robot>

File: src/my_robot_description/models/my_robot_description/my_robot_core.xacro (robot description, xacro)
@@ -36,5 +36,5 @@
       <origin xyz="0 0 0" rpy="0 0 0"/>
       <geometry>
-        <mesh filename="file://$(find my_robot_description)/models/my_robot_description/meshes/base_link.STL"/>
+        <mesh filename="file://$(find my_robot_description)/models/my_robot_description/meshes/base_link.stl"/>
       </geometry>
       <material name="">
@@ -45,5 +45,5 @@
       <origin xyz="0 0 0" rpy="0 0 0"/>
       <geometry>
-        <mesh filename="file://$(find my_robot_description)/models/my_robot_description/meshes/base_link.STL"/>
+        <mesh filename="file://$(find my_robot_description)/models/my_robot_description/meshes/base_link.stl"/>
       </geometry>
     </collision>
@@ -93,12 +93,12 @@
       <origin xyz="0 0 0" rpy="0 0 0"/>
       <geometry>
-        <mesh filename="file://$(find my_robot_description)/models/my_robot_description/meshes/BL_link.STL"/>
-      </geometry>
-      <material name=""><color rgba="0.79216 0.81961 0.93333 1"/></material>
-    </visual>
-    <collision>
-      <origin xyz="0 0 0" rpy="0 0 0"/>
-      <geometry>
-        <mesh filename="file://$(find my_robot_description)/models/my_robot_description/meshes/BL_link.STL"/>
+        <mesh filename="file://$(find my_robot_description)/models/my_robot_description/meshes/BL_link.stl"/>
+      </geometry>
+      <material name=""><color rgba="0.79216 0.81961 0.93333 1"/></material>
+    </visual>
+    <collision>
+      <origin xyz="0 0 0" rpy="0 0 0"/>
+      <geometry>
+        <mesh filename="file://$(find my_robot_description)/models/my_robot_description/meshes/BL_link.stl"/>
       </geometry>
     </collision>
@@ -117,12 +117,12 @@
       <origin xyz="0 0 0" rpy="0 0 0"/>
       <geometry>
-        <mesh filename="file://$(find my_robot_description)/models/my_robot_description/meshes/BR_link.STL"/>
-      </geometry>
-      <material name=""><color rgba="0.79216 0.81961 0.93333 1"/></material>
-    </visual>
-    <collision>
-      <origin xyz="0 0 0" rpy="0 0 0"/>
-      <geometry>
-        <mesh filename="file://$(find my_robot_description)/models/my_robot_description/meshes/BR_link.STL"/>
+        <mesh filename="file://$(find my_robot_description)/models/my_robot_description/meshes/BR_link.stl"/>
+      </geometry>
+      <material name=""><color rgba="0.79216 0.81961 0.93333 1"/></material>
+    </visual>
+    <collision>
+      <origin xyz="0 0 0" rpy="0 0 0"/>
+      <geometry>
+        <mesh filename="file://$(find my_robot_description)/models/my_robot_description/meshes/BR_link.stl"/>
       </geometry>
     </collision>
@@ -141,12 +141,12 @@
       <origin xyz="0 0 0" rpy="0 0 0"/>
       <geometry>
-        <mesh filename="file://$(find my_robot_description)/models/my_robot_description/meshes/FL_link.STL"/>
-      </geometry>
-      <material name=""><color rgba="0.79216 0.81961 0.93333 1"/></material>
-    </visual>
-    <collision>
-      <origin xyz="0 0 0" rpy="0 0 0"/>
-      <geometry>
-        <mesh filename="file://$(find my_robot_description)/models/my_robot_description/meshes/FL_link.STL"/>
+        <mesh filename="file://$(find my_robot_description)/models/my_robot_description/meshes/FL_link.stl"/>
+      </geometry>
+      <material name=""><color rgba="0.79216 0.81961 0.93333 1"/></material>
+    </visual>
+    <collision>
+      <origin xyz="0 0 0" rpy="0 0 0"/>
+      <geometry>
+        <mesh filename="file://$(find my_robot_description)/models/my_robot_description/meshes/FL_link.stl"/>
       </geometry>
     </collision>
@@ -165,12 +165,12 @@
       <origin xyz="0 0 0" rpy="0 0 0"/>
       <geometry>
-        <mesh filename="file://$(find my_robot_description)/models/my_robot_description/meshes/FR_link.STL"/>
-      </geometry>
-      <material name=""><color rgba="0.79216 0.81961 0.93333 1"/></material>
-    </visual>
-    <collision>
-      <origin xyz="0 0 0" rpy="0 0 0"/>
-      <geometry>
-        <mesh filename="file://$(find my_robot_description)/models/my_robot_description/meshes/FR_link.STL"/>
+        <mesh filename="file://$(find my_robot_description)/models/my_robot_description/meshes/FR_link.stl"/>
+      </geometry>
+      <material name=""><color rgba="0.79216 0.81961 0.93333 1"/></material>
+    </visual>
+    <collision>
+      <origin xyz="0 0 0" rpy="0 0 0"/>
+      <geometry>
+        <mesh filename="file://$(find my_robot_description)/models/my_robot_description/meshes/FR_link.stl"/>
       </geometry>
     </collision>
